File: Hardware/LilyTiny.brd (EAGLE design)
At the start: 20 x 20 mm, 13 parts, among them U1 ATTINY85

Commit message: Fixing merge conflicts numero dos.
Getting files ready for production runs.
Parts:
- added FRAME2: FRAME-LETTER, SparkFun-Aesthetics:CREATIVE_COMMONS
- added LOGO1: OSHW-LOGOS, SparkFun-Aesthetics:OSHW-LOGO-S
- added LOGO2: SFE_LOGO_FLAME.1_INCH, SparkFun-Aesthetics:SFE_LOGO_FLAME_.1
- C1: device SparkFun:0402-CAP -> SparkFun:0603-CAP
- R1: device SparkFun:0402-RES -> SparkFun:0603-RES
- U$1: value CREATIVE_COMMONS -> REVISION; device SparkFun:CREATIVE_COMMONS -> SparkFun-Aesthetics:REVISION
- moved U$1 26.7 mm to (-15.2, -22.9)
- moved C1 2.18 mm to (1.78, 3.81), turned to 0 degrees
- moved R1 1.78 mm to (-1.78, 3.81)
Routing:
- net N$9: track 4.86 -> 0.00 mm, vias 1 -> 0
- net N$4: track 10.3 -> 14.0 mm, vias 0 -> 2
- net VCC: track 16.8 -> 14.0 mm
- net NRESET: track 12.0 -> 14.1 mm
- net N$3: vias 0 -> 1
- net N$5: vias 0 -> 1
Other:
- board text added: "P. Lewis, T. Klopfenstein"
- board text added: "Tiny"
- board text added: "Twinkle"
- board text added: "v12"

Commit message: Added regular fid to board. Deleted old gerbs
Parts:
- removed JP1, JP2: FIDUCIALUFIDUCIAL, SparkFun:MICRO-FIDUCIAL
- added FID1, FID2: FIDUCIAL1X2, SparkFun-Aesthetics:FIDUCIAL-1X2
