File: Hardware/LilyTiny.brd (EAGLE design)
At the start: 20 x 20 mm, 16 parts, among them U1 ATTINY85

Commit message: Switched programming lines from vias to device
-Used AVR_SPI_PRG_6.dev with the new "TEST_POINTS" package (which
include the necessary stop mask).

-Centered symbols in schematic.
Parts:
- added J1: (no value), SparkFun-Connectors:2X3_TEST_POINTS
Connections:
- removed net N$3: U$7.1, U1.5
- removed net N$4: U$3.1, U1.6
- removed net N$5: U$4.1, U1.7
- new net MISO: J1.1, U$3.1, U1.6
- new net MOSI: J1.4, U$7.1, U1.5
- new net SCK: J1.3, U$4.1, U1.7
- net GND: now also J1.6
- net NRESET: now also J1.5
- net VCC: now also J1.2
Routing:
- net N$4: track 14.0 -> 0.00 mm, vias 2 -> 0
- net MISO: track 0.00 -> 14.0 mm, vias 0 -> 1
- net N$3: track 12.8 -> 0.00 mm, vias 1 -> 0
- net MOSI: track 0.00 -> 12.8 mm
- net SCK: track 0.00 -> 8.15 mm
- net N$5: track 8.15 -> 0.00 mm, vias 1 -> 0
- net VCC: vias 1 -> 0
- net NRESET: vias 2 -> 1
Other:
- board text added: "v13"
- board text removed: "v12"
