File: Production Files/LilyTiny-Panel-v12.brd (EAGLE design)
At the start: 114.8 x 114.8 mm, 353 parts, among them U1 ATTINY85, U10 ATTINY85, U11 ATTINY85, U12 ATTINY85, U13 ATTINY85, U14 ATTINY85, U15 ATTINY85, U16 ATTINY85, U17 ATTINY85, U18 ATTINY85, U19 ATTINY85, U2 ATTINY85, U20 ATTINY85, U21 ATTINY85, U22 ATTINY85, U23 ATTINY85, U24 ATTINY85, U25 ATTINY85, U3 ATTINY85, U4 ATTINY85, U5 ATTINY85, U6 ATTINY85, U7 ATTINY85, U8 ATTINY85, U9 ATTINY85

Commit message: re-did panel v12
Parts:
- removed E$5: (no value), SparkFun-Aesthetics:FIDUCIAL-1X2
- added E$6: (no value), SparkFun-Aesthetics:FIDUCIAL-1X2
- added J1, J10, J11, J12, J13, J14, J15, J16, J17, J18, J19, J2, J20, J21, J22, J23, J24, J25, J3, J4, J5, J6, J7, J8, J9: (no value), SparkFun-Connectors:2X3_TEST_POINTS
- moved E$1 0.76 mm to (4.57, 11.4)
- moved E$4 0.25 mm to (110.4, 11.7)
Connections:
- removed net N$10 (its old number): U$20.1, U3.5
- removed net N$100: U$171.1, U25.7
- removed net N$11 (its old number): U$16.1, U3.6
- removed net N$12 (its old number): U$17.1, U3.7
- removed net N$14 (its old number): U$27.1, U4.5
- removed net N$15 (its old number): U$23.1, U4.6
- removed net N$16 (its old number): U$24.1, U4.7
- removed net N$18 (its old number): U$34.1, U5.5
- removed net N$19 (its old number): U$30.1, U5.6
- removed net N$2 (its old number): U$13.1, U2.5
- removed net N$20 (its old number): U$31.1, U5.7
- removed net N$22 (its old number): U$41.1, U6.5
- removed net N$23 (its old number): U$37.1, U6.6
- removed net N$24 (its old number): U$38.1, U6.7
- removed net N$26 (its old number): U$48.1, U7.5
- removed net N$27: U$44.1, U7.6
- removed net N$28: U$45.1, U7.7
- removed net N$3 (its old number): U$7.1, U1.5
- removed net N$30: U$55.1, U8.5
- removed net N$31: U$51.1, U8.6
- removed net N$32: U$52.1, U8.7
- removed net N$34: U$62.1, U9.5
- removed net N$35: U$58.1, U9.6
- removed net N$36: U$59.1, U9.7
- removed net N$38: U$69.1, U10.5
- removed net N$39: U$65.1, U10.6
- removed net N$4 (its old number): U$3.1, U1.6
- removed net N$40: U$66.1, U10.7
- removed net N$42: U$76.1, U11.5
- removed net N$43: U$72.1, U11.6
- removed net N$44: U$73.1, U11.7
- removed net N$46: U$83.1, U12.5
- removed net N$47: U$79.1, U12.6
- removed net N$48: U$80.1, U12.7
- removed net N$5 (its old number): U$4.1, U1.7
- removed net N$50: U$90.1, U13.5
- removed net N$51: U$86.1, U13.6
- removed net N$52: U$87.1, U13.7
- removed net N$54: U$97.1, U14.5
- removed net N$55: U$93.1, U14.6
- removed net N$56: U$94.1, U14.7
- removed net N$58: U$104.1, U15.5
- removed net N$59: U$100.1, U15.6
- removed net N$60: U$101.1, U15.7
- removed net N$62: U$111.1, U16.5
- removed net N$63: U$107.1, U16.6
- removed net N$64: U$108.1, U16.7
- removed net N$66: U$118.1, U17.5
- removed net N$67: U$114.1, U17.6
- removed net N$68: U$115.1, U17.7
- removed net N$7 (its old number): U$9.1, U2.6
- removed net N$70: U$125.1, U18.5
- removed net N$71: U$121.1, U18.6
- removed net N$72: U$122.1, U18.7
- removed net N$74: U$132.1, U19.5
- removed net N$75: U$128.1, U19.6
- removed net N$76: U$129.1, U19.7
- removed net N$78: U$139.1, U20.5
- removed net N$79: U$135.1, U20.6
- removed net N$8 (its old number): U$10.1, U2.7
- removed net N$80: U$136.1, U20.7
- removed net N$82: U$146.1, U21.5
- removed net N$83: U$142.1, U21.6
- removed net N$84: U$143.1, U21.7
- removed net N$86: U$153.1, U22.5
- removed net N$87: U$149.1, U22.6
- removed net N$88: U$150.1, U22.7
- removed net N$90: U$160.1, U23.5
- removed net N$91: U$156.1, U23.6
- removed net N$92: U$157.1, U23.7
- removed net N$94: U$167.1, U24.5
- removed net N$95: U$163.1, U24.6
- removed net N$96: U$164.1, U24.7
- removed net N$98: U$174.1, U25.5
- removed net N$99: U$170.1, U25.6
- new net MISO: J1.1, U$3.1, U1.6
- new net MISO1: J2.1, U$9.1, U2.6
- new net MISO10: J11.1, U$72.1, U11.6
- new net MISO11: J12.1, U$79.1, U12.6
- new net MISO12: J13.1, U$86.1, U13.6
- new net MISO13: J14.1, U$93.1, U14.6
- new net MISO14: J15.1, U$100.1, U15.6
- new net MISO15: J16.1, U$107.1, U16.6
- new net MISO16: J17.1, U$114.1, U17.6
- new net MISO17: J18.1, U$121.1, U18.6
- new net MISO18: J19.1, U$128.1, U19.6
- new net MISO19: J20.1, U$135.1, U20.6
- new net MISO2: J3.1, U$16.1, U3.6
- new net MISO20: J21.1, U$142.1, U21.6
- new net MISO21: J22.1, U$149.1, U22.6
- new net MISO22: J23.1, U$156.1, U23.6
- new net MISO23: J24.1, U$163.1, U24.6
- new net MISO24: J25.1, U$170.1, U25.6
- new net MISO3: J4.1, U$23.1, U4.6
- new net MISO4: J5.1, U$30.1, U5.6
- new net MISO5: J6.1, U$37.1, U6.6
- new net MISO6: J7.1, U$44.1, U7.6
- new net MISO7: J8.1, U$51.1, U8.6
- new net MISO8: J9.1, U$58.1, U9.6
- new net MISO9: J10.1, U$65.1, U10.6
- new net MOSI: J1.4, U$7.1, U1.5
- new net MOSI1: J2.4, U$13.1, U2.5
- new net MOSI10: J11.4, U$76.1, U11.5
- new net MOSI11: J12.4, U$83.1, U12.5
- new net MOSI12: J13.4, U$90.1, U13.5
- new net MOSI13: J14.4, U$97.1, U14.5
- new net MOSI14: J15.4, U$104.1, U15.5
- new net MOSI15: J16.4, U$111.1, U16.5
- new net MOSI16: J17.4, U$118.1, U17.5
- new net MOSI17: J18.4, U$125.1, U18.5
- new net MOSI18: J19.4, U$132.1, U19.5
- new net MOSI19: J20.4, U$139.1, U20.5
- new net MOSI2: J3.4, U$20.1, U3.5
- new net MOSI20: J21.4, U$146.1, U21.5
- new net MOSI21: J22.4, U$153.1, U22.5
- new net MOSI22: J23.4, U$160.1, U23.5
- new net MOSI23: J24.4, U$167.1, U24.5
- new net MOSI24: J25.4, U$174.1, U25.5
- new net MOSI3: J4.4, U$27.1, U4.5
- new net MOSI4: J5.4, U$34.1, U5.5
- new net MOSI5: J6.4, U$41.1, U6.5
- new net MOSI6: J7.4, U$48.1, U7.5
- new net MOSI7: J8.4, U$55.1, U8.5
- new net MOSI8: J9.4, U$62.1, U9.5
- new net MOSI9: J10.4, U$69.1, U10.5
- new net SCK: J1.3, U$4.1, U1.7
- new net SCK1: J2.3, U$10.1, U2.7
- new net SCK10: J11.3, U$73.1, U11.7
- new net SCK11: J12.3, U$80.1, U12.7
- new net SCK12: J13.3, U$87.1, U13.7
- new net SCK13: J14.3, U$94.1, U14.7
- new net SCK14: J15.3, U$101.1, U15.7
- new net SCK15: J16.3, U$108.1, U16.7
- new net SCK16: J17.3, U$115.1, U17.7
- new net SCK17: J18.3, U$122.1, U18.7
- new net SCK18: J19.3, U$129.1, U19.7
- new net SCK19: J20.3, U$136.1, U20.7
- new net SCK2: J3.3, U$17.1, U3.7
- new net SCK20: J21.3, U$143.1, U21.7
- new net SCK21: J22.3, U$150.1, U22.7
- new net SCK22: J23.3, U$157.1, U23.7
- new net SCK23: J24.3, U$164.1, U24.7
- new net SCK24: J25.3, U$171.1, U25.7
- new net SCK3: J4.3, U$24.1, U4.7
- new net SCK4: J5.3, U$31.1, U5.7
- new net SCK5: J6.3, U$38.1, U6.7
- new net SCK6: J7.3, U$45.1, U7.7
- new net SCK7: J8.3, U$52.1, U8.7
- new net SCK8: J9.3, U$59.1, U9.7
- new net SCK9: J10.3, U$66.1, U10.7
- net GND: now also J1.6
- net GND1: now also J2.6
- net GND10: now also J11.6
- net GND11: now also J12.6
- net GND12: now also J13.6
- net GND13: now also J14.6
- net GND14: now also J15.6
- net GND15: now also J16.6
- net GND16: now also J17.6
- net GND17: now also J18.6
- net GND18: now also J19.6
- net GND19: now also J20.6
- net GND2: now also J3.6
- net GND20: now also J21.6
- net GND21: now also J22.6
- net GND22: now also J23.6
- net GND23: now also J24.6
- net GND24: now also J25.6
- net GND3: now also J4.6
- net GND4: now also J5.6
- net GND5: now also J6.6
- net GND6: now also J7.6
- net GND7: now also J8.6
- net GND8: now also J9.6
- net GND9: now also J10.6
- net NRESET: now also J1.5
- net NRESET1: now also J2.5
- net NRESET10: now also J11.5
- net NRESET11: now also J12.5
- net NRESET12: now also J13.5
- net NRESET13: now also J14.5
- net NRESET14: now also J15.5
- net NRESET15: now also J16.5
- net NRESET16: now also J17.5
- net NRESET17: now also J18.5
- net NRESET18: now also J19.5
- net NRESET19: now also J20.5
- net NRESET2: now also J3.5
- net NRESET20: now also J21.5
- net NRESET21: now also J22.5
- net NRESET22: now also J23.5
- net NRESET23: now also J24.5
- net NRESET24: now also J25.5
- net NRESET3: now also J4.5
- net NRESET4: now also J5.5
- net NRESET5: now also J6.5
- net NRESET6: now also J7.5
- net NRESET7: now also J8.5
- net NRESET8: now also J9.5
- net NRESET9: now also J10.5
- net VCC: now also J1.2
- net VCC1: now also J2.2
- net VCC10: now also J11.2
- net VCC11: now also J12.2
- net VCC12: now also J13.2
- net VCC13: now also J14.2
- net VCC14: now also J15.2
- net VCC15: now also J16.2
- net VCC16: now also J17.2
- net VCC17: now also J18.2
- net VCC18: now also J19.2
- net VCC19: now also J20.2
- net VCC2: now also J3.2
- net VCC20: now also J21.2
- net VCC21: now also J22.2
- net VCC22: now also J23.2
- net VCC23: now also J24.2
- net VCC24: now also J25.2
- net VCC3: now also J4.2
- net VCC4: now also J5.2
- net VCC5: now also J6.2
- net VCC6: now also J7.2
- net VCC7: now also J8.2
- net VCC8: now also J9.2
- net VCC9: now also J10.2
Routing:
- net N$95: track 14.0 -> 0.00 mm, vias 2 -> 0
- net MISO23: track 0.00 -> 14.0 mm, vias 0 -> 1
- net N$83: track 14.0 -> 0.00 mm, vias 2 -> 0
- net MISO20: track 0.00 -> 14.0 mm, vias 0 -> 1
- net N$55: track 14.0 -> 0.00 mm, vias 2 -> 0
- net N$35: track 14.0 -> 0.00 mm, vias 2 -> 0
- net MISO8: track 0.00 -> 14.0 mm, vias 0 -> 1
- net MISO13: track 0.00 -> 14.0 mm, vias 0 -> 1
- net N$75: track 14.0 -> 0.00 mm, vias 2 -> 0
- net MISO18: track 0.00 -> 14.0 mm, vias 0 -> 1
- net N$15 (its old number): track 14.0 -> 0.00 mm, vias 2 -> 0
- net MISO3: track 0.00 -> 14.0 mm, vias 0 -> 1
- net N$99: track 14.0 -> 0.00 mm, vias 2 -> 0
- net N$43: track 14.0 -> 0.00 mm, vias 2 -> 0
- net N$23 (its old number): track 14.0 -> 0.00 mm, vias 2 -> 0
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Other:
- outline, holes or cut-outs redrawn
- board text added: "v13"
- board text removed: "v12"
